Commit message: GP12-Meshes-Update
Updated visual mesh from .stl to .dae
Updated xacro file to newer format with flange and tool0

File: motoman_gp12_support/urdf/gp12_macro.xacro (robot description, xacro)
@@ -7,5 +7,5 @@
         <visual>
             <geometry>
-                <mesh filename="package://motoman_gp12_support/meshes/visual/gp12_base_link.stl"/>
+                <mesh filename="package://motoman_gp12_support/meshes/visual/gp12_base_link.dae"/>
             </geometry>
             <xacro:material_yaskawa_blue/>
@@ -20,5 +20,5 @@
         <visual>
             <geometry>
-                <mesh filename="package://motoman_gp12_support/meshes/visual/gp12_link_1_s.stl"/>
+                <mesh filename="package://motoman_gp12_support/meshes/visual/gp12_link_1_s.dae"/>
             </geometry>
             <xacro:material_yaskawa_blue/>
@@ -33,5 +33,5 @@
         <visual>
             <geometry>
-                <mesh filename="package://motoman_gp12_support/meshes/visual/gp12_link_2_l.stl"/>
+                <mesh filename="package://motoman_gp12_support/meshes/visual/gp12_link_2_l.dae"/>
             </geometry>
             <xacro:material_yaskawa_blue/>
@@ -46,5 +46,5 @@
         <visual>
             <geometry>
-                <mesh filename="package://motoman_gp12_support/meshes/visual/gp12_link_3_u.stl"/>
+                <mesh filename="package://motoman_gp12_support/meshes/visual/gp12_link_3_u.dae"/>
             </geometry>
             <xacro:material_yaskawa_blue/>
@@ -59,5 +59,5 @@
         <visual>
             <geometry>
-                <mesh filename="package://motoman_gp12_support/meshes/visual/gp12_link_4_r.stl"/>
+                <mesh filename="package://motoman_gp12_support/meshes/visual/gp12_link_4_r.dae"/>
             </geometry>
             <xacro:material_yaskawa_blue/>
@@ -72,5 +72,5 @@
         <visual>
             <geometry>
-                <mesh filename="package://motoman_gp12_support/meshes/visual/gp12_link_5_b.stl"/>
+                <mesh filename="package://motoman_gp12_support/meshes/visual/gp12_link_5_b.dae"/>
             </geometry>
             <xacro:material_yaskawa_blue/>
@@ -85,5 +85,5 @@
         <visual>
             <geometry>
-                <mesh filename="package://motoman_gp12_support/meshes/visual/gp12_link_6_t.stl"/>
+                <mesh filename="package://motoman_gp12_support/meshes/visual/gp12_link_6_t.dae"/>
             </geometry>
             <xacro:material_yaskawa_blue/>
@@ -140,9 +140,4 @@
         <limit lower="-7.9412" upper="7.9412" effort="33.30" velocity="12.2143"/>
     </joint>
-    <joint name="${prefix}joint_6_t-tool0" type="fixed">
-        <origin xyz="0.100 0 0" rpy="3.1415926 -1.570796 0"/>
-        <parent link="${prefix}link_6_t"/>
-        <child link="${prefix}tool0"/>
-    </joint>
     <!-- end of joint list -->
     <!-- ROS base_link to Robot Manufacturer World Coordinates transform -->
@@ -153,4 +148,18 @@
         <child link="${prefix}base"/>
     </joint>
+    <!-- ROS-Industrial 'flange' frame: attachment point for EEF models -->
+    <link name="${prefix}flange" />
+    <joint name="${prefix}joint_6_t-flange" type="fixed">
+        <origin xyz="0.100 0 0" rpy="0 0 0" />
+        <parent link="${prefix}link_6_t" />
+        <child link="${prefix}flange" />
+    </joint>
+    <!-- ROS-Industrial 'tool0' frame: all-zeros tool frame -->
+    <link name="${prefix}tool0" />
+    <joint name="${prefix}flange-tool0" type="fixed">
+        <origin xyz="0 0 0" rpy="${radians(180)} ${radians(-90)} 0" />
+        <parent link="${prefix}flange" />
+        <child link="${prefix}tool0" />
+    </joint>
     </xacro:macro>
 </robot>

Commit message: Fix error in model
There was a 3 mm error in the models Z position that was fixed
Changed model 6_t to full plate instead of only ring
Generated t-axis cavity on model 5_b

File: motoman_gp12_support/urdf/gp12_macro.xacro (robot description, xacro)
@@ -95,5 +95,4 @@
         </collision>
     </link>
-    <link name="${prefix}tool0"/>
     <!-- end of link list -->
     <!-- joint list -->
